File: Functional Test/Ki-Test 01-09 - Backup/Diodes.kicad_sch (KiCad schematic)
At the start: 6 parts

Commit message: oclean up graphics and added some bling and trying to work with kiCad restore
Parts:
- D1, D2, D3, D4, D5, D6: symbol Diode:1N4004 -> MySymbols:1N4004
Changed lines of the file:
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@@
 	)
 	(symbol
-		(lib_id "Diode:1N4004")
+		(lib_id "MySymbols:1N4004")
 		(at 133.35 73.66 270)
 		(unit 1)
@@
 			)
 		)
-		(property "Datasheet" "http://www.vishay.com/docs/88503/1n4001.pdf"
+		(property "Datasheet" "https://diotec.com/request/datasheet/1n4001.pdf"
 			(at 133.35 73.66 0)
 			(effects
@@
 	)
 	(symbol
-		(lib_id "Diode:1N4004")
+		(lib_id "MySymbols:1N4004")
 		(at 133.35 95.25 270)
 		(unit 1)
@@
 			)
 		)
-		(property "Datasheet" "http://www.vishay.com/docs/88503/1n4001.pdf"
+		(property "Datasheet" "https://diotec.com/request/datasheet/1n4001.pdf"
 			(at 133.35 95.25 0)
 			(effects
@@
 	)
 	(symbol
-		(lib_id "Diode:1N4004")
+		(lib_id "MySymbols:1N4004")
 		(at 144.78 73.66 270)
 		(unit 1)
@@
 			)
 		)
-		(property "Datasheet" "http://www.vishay.com/docs/88503/1n4001.pdf"
+		(property "Datasheet" "https://diotec.com/request/datasheet/1n4001.pdf"
 			(at 144.78 73.66 0)
 			(effects
@@
 	)
 	(symbol
-		(lib_id "Diode:1N4004")
+		(lib_id "MySymbols:1N4004")
 		(at 144.78 95.25 270)
 		(unit 1)
@@
 			)
 		)
-		(property "Datasheet" "http://www.vishay.com/docs/88503/1n4001.pdf"
+		(property "Datasheet" "https://diotec.com/request/datasheet/1n4001.pdf"
 			(at 144.78 95.25 0)
 			(effects
@@
 	)
 	(symbol
-		(lib_id "Diode:1N4004")
+		(lib_id "MySymbols:1N4004")
 		(at 156.21 95.25 270)
 		(unit 1)
@@
 			)
 		)
-		(property "Datasheet" "http://www.vishay.com/docs/88503/1n4001.pdf"
+		(property "Datasheet" "https://diotec.com/request/datasheet/1n4001.pdf"
 			(at 156.21 95.25 0)
 			(effects
@@
 	)
 	(symbol
-		(lib_id "Diode:1N4004")
+		(lib_id "MySymbols:1N4004")
 		(at 156.21 73.66 270)
 		(unit 1)
@@
 			)
 		)
-		(property "Datasheet" "http://www.vishay.com/docs/88503/1n4001.pdf"
+		(property "Datasheet" "https://diotec.com/request/datasheet/1n4001.pdf"
 			(at 156.21 73.66 0)
 			(effects
