File: Functional Test/Ki-Test 01-09 - Backup/Ki-Test.kicad_pcb (KiCad board)
At the start: 2 copper layers, 32 parts, among them J1 Conn_01x01

Commit message: oclean up graphics and added some bling and trying to work with kiCad restore
Parts:
- removed REF**: KSA_Tactile_SPST, Button_Switch_THT:KSA_Tactile_SPST
- J1: footprint Connector_Phoenix_MC:PhoenixContact_MCV_1,5_4-GF-3.5_1x04_P3.50mm_Vertical_ThreadedFlange -> Connector_Phoenix_MC:PhoenixContact_MCV_1,5_4-GF-3.5_1x04_P3.50mm_Vertical_ThreadedFlange_MountHole
- moved D7 76.4 mm to (137.4, 117.3)
- moved J1 69.7 mm to (73.9, 68.3)
- moved D3 47.7 mm to (137.4, 123.5)
- moved D13 35.8 mm to (137.4, 129.8)
- moved C1 29.8 mm to (95.3, 55.6)
- moved C2 29.8 mm to (95.3, 76.1)
- moved C3 29.8 mm to (95.3, 96.7)
- moved D14 17.1 mm to (137.4, 93.9)
- moved D15 17.1 mm to (137.4, 98.2)
- moved D16 17.1 mm to (137.4, 102.4)
- moved D17 17.1 mm to (137.4, 106.7)
- moved D18 17.1 mm to (137.4, 110.9)
- moved R2 15.7 mm to (120.3, 55.9)
- moved R3 15.7 mm to (120.3, 62.7)
- moved R4 15.7 mm to (120.3, 69.6)
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