File: Functional Test/Ki-Test 01-09 - Backup/Ki-Test.kicad_sch (KiCad schematic)
At the start: 14 parts, among them J1 Conn_01x01

Commit message: oclean up graphics and added some bling and trying to work with kiCad restore
Parts:
- C1, C2, C3: symbol Device:C_US -> MySymbols:C_US
- J1: footprint Connector_Phoenix_MC:PhoenixContact_MCV_1,5_4-GF-3.5_1x04_P3.50mm_Vertical_ThreadedFlange -> (none); symbol Connector_Generic:Conn_01x04 -> MySymbols:Conn_01x04
- R1, R2, R3, R4, R5, R6, R7, R8, R9: symbol Device:R -> MySymbols:R
- R10: footprint (none) -> Resistor_SMD:R_4020_10251Metric_Pad1.65x5.30mm_HandSolder; symbol Device:R -> MySymbols:R
Changed lines of the file:
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@@
 	)
 	(symbol
-		(lib_id "Device:R")
+		(lib_id "MySymbols:R")
 		(at 139.7 66.04 90)
 		(unit 1)
@@
 			)
 		)
-		(property "Datasheet" "https://yageogroup.com/content/datasheet/asset/file/PYU-RC_GROUP_51_ROHS_L"
+		(property "Datasheet" "https://www.digikey.com/en/models/462974"
 			(at 139.7 66.04 0)
 			(effects
@@
 	)
 	(symbol
-		(lib_id "Device:R")
+		(lib_id "MySymbols:R")
 		(at 139.7 71.12 90)
 		(unit 1)
@@
 			)
 		)
-		(property "Datasheet" "https://yageogroup.com/content/datasheet/asset/file/PYU-RC_GROUP_51_ROHS_L"
+		(property "Datasheet" "https://www.digikey.com/en/models/462974"
 			(at 139.7 71.12 0)
 			(effects
@@
 	)
 	(symbol
-		(lib_id "Device:R")
+		(lib_id "MySymbols:R")
 		(at 139.7 93.98 90)
 		(unit 1)
@@
 			)
 		)
-		(property "Datasheet" "https://www.seielect.com/catalog/SEI-CF_CFM.pdf"
+		(property "Datasheet" "https://www.digikey.com/en/models/462974"
 			(at 139.7 93.98 0)
 			(effects
@@
 	)
 	(symbol
-		(lib_id "Device:R")
+		(lib_id "MySymbols:R")
 		(at 139.7 57.15 90)
 		(unit 1)
@@
 			)
 		)
-		(property "Footprint" ""
+		(property "Footprint" "Resistor_SMD:R_4020_10251Metric_Pad1.65x5.30mm_HandSolder"
 			(at 139.7 58.928 90)
 			(effects
@@
 			)
 		)
-		(property "Datasheet" "https://www.koaspeer.com/pdfs/RC.pdf"
+		(property "Datasheet" "https://www.digikey.com/en/models/462974"
 			(at 139.7 57.15 0)
 			(effects
@@
 	)
 	(symbol
-		(lib_id "Device:C_US")
+		(lib_id "MySymbols:C_US")
 		(at 174.0027 71.12 0)
 		(unit 1)
@@
 	)
 	(symbol
-		(lib_id "Device:R")
+		(lib_id "MySymbols:R")
 		(at 139.7 111.76 90)
 		(unit 1)
@@
 			)
 		)
-		(property "Datasheet" "https://www.ohmite.com/assets/images/res-ox-oy-rev-7.23.pdf"
+		(property "Datasheet" "https://www.digikey.com/en/models/462974"
 			(at 139.7 111.76 0)
 			(effects
@@
 	)
 	(symbol
-		(lib_id "Device:R")
+		(lib_id "MySymbols:R")
 		(at 139.7 88.9 90)
 		(unit 1)
@@
 			)
 		)
-		(property "Datasheet" "https://www.seielect.com/catalog/SEI-CF_CFM.pdf"
+		(property "Datasheet" "https://www.digikey.com/en/models/462974"
 			(at 139.7 88.9 0)
 			(effects
@@
 	)
 	(symbol
-		(lib_id "Connector_Generic:Conn_01x04")
+		(lib_id "MySymbols:Conn_01x04")
 		(at 91.44 68.58 0)
 		(mirror y)
@@
 			)
 		)
-		(property "Footprint" "Connector_Phoenix_MC:PhoenixContact_MCV_1,5_4-GF-3.5_1x04_P3.50mm_Vertical_ThreadedFlange"
+		(property "Footprint" ""
 			(at 91.44 68.58 0)
 			(effects
@@
 			)
 		)
-		(property "Datasheet" "~"
+		(property "Datasheet" "http://www.phoenixcontact.com/us/products/1843240/pdf"
 			(at 91.44 68.58 0)
 			(effects
@@
 	)
 	(symbol
-		(lib_id "Device:R")
+		(lib_id "MySymbols:R")
 		(at 139.7 121.92 90)
 		(unit 1)
@@
 			)
 		)
-		(property "Datasheet" "https://www.digikey.com/en/models/823904?tab=ultralibrarian"
+		(property "Datasheet" "https://www.digikey.com/en/models/462974"
 			(at 139.7 121.92 0)
 			(effects
@@
 	)
 	(symbol
-		(lib_id "Device:R")
+		(lib_id "MySymbols:R")
 		(at 139.7 76.2 90)
 		(unit 1)
@@
 			)
 		)
-		(property "Datasheet" "https://yageogroup.com/content/datasheet/asset/file/PYU-RC_GROUP_51_ROHS_L"
+		(property "Datasheet" "https://www.digikey.com/en/models/462974"
 			(at 139.7 76.2 0)
 			(effects
@@
 	)
 	(symbol
-		(lib_id "Device:R")
+		(lib_id "MySymbols:R")
 		(at 139.7 99.06 90)
 		(unit 1)
@@
 			)
 		)
-		(property "Datasheet" "https://www.seielect.com/catalog/SEI-CF_CFM.pdf"
+		(property "Datasheet" "https://www.digikey.com/en/models/462974"
 			(at 139.7 99.06 0)
 			(effects
@@
 	)
 	(symbol
-		(lib_id "Device:C_US")
+		(lib_id "MySymbols:C_US")
 		(at 173.99 93.98 0)
 		(unit 1)
@@
 	)
 	(symbol
-		(lib_id "Device:R")
+		(lib_id "MySymbols:R")
 		(at 139.7 116.84 90)
 		(unit 1)
@@
 			)
 		)
-		(property "Datasheet" "https://www.ohmite.com/assets/images/res-ox-oy-rev-7.23.pdf"
+		(property "Datasheet" "https://www.digikey.com/en/models/462974"
 			(at 139.7 116.84 0)
 			(effects
@@
 	)
 	(symbol
-		(lib_id "Device:C_US")
+		(lib_id "MySymbols:C_US")
 		(at 173.99 116.84 0)
 		(unit 1)
